File: FreePillV1.0.kicad_sch (KiCad schematic)
At the start: 11 parts

Commit message: last commit failed
Connections:
- net GND: no longer C?.1, C?.2, C?.2
- new net: C?.1, C?.2, C?.2
Changed lines of the file:
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@@
     (pin "2")
-  )
-  (symbol (lib_id "power:GND") (at 135.89 45.72 0) (unit 1)
-    (in_bom yes) (on_board yes) (fields_autoplaced)
-    (property "Reference" "#PWR?" (id 0) (at 135.89 52.07 0)
-      (effects (font (size 1.27 1.27)) hide)
-    )
-    (property "Value" "GND" (id 1) (at 135.89 50.8 0))
-    (property "Footprint" "" (id 2) (at 135.89 45.72 0)
-      (effects (font (size 1.27 1.27)) hide)
-    )
-    (property "Datasheet" "" (id 3) (at 135.89 45.72 0)
-      (effects (font (size 1.27 1.27)) hide)
-    )
-    (pin "1")
   )
   (symbol (lib_id "Device:C_Small") (at 124.46 54.61 270) (unit 1)
@@
       (reference "#PWR?") (unit 1) (value "GND") (footprint "")
     )
-    (path "/d799a517-6629-4915-9e9e-a928069731d8"
-      (reference "#PWR?") (unit 1) (value "GND") (footprint "")
-    )

Commit message: Completed the following:
-decoupling caps
-reset and boot mode circuits
-arrangement (bounding boxes) of completed circuits
Parts:
- removed C? (x5): 100n, Capacitor_SMD:C_0402_1005Metric_Pad0.74x0.62mm_HandSolder, symbol Device:C_Small
- removed C?: 2.2u, Capacitor_SMD:C_0603_1608Metric_Pad1.08x0.95mm_HandSolder, symbol Device:C_Small
- added C? (x6): 100nF, symbol Device:C_Small
- added C?: 2.2u, Capacitor_SMD:C_0603_1608Metric_Pad1.08x0.95mm_HandSolder, symbol Device:C_Small
- added C?: 2.2uF, symbol Device:C_Small
- added R? (x2): 10k, symbol Device:R_Small
- added SW? (x2): SW_Push, symbol Switch:SW_Push
Connections:
- net +3V3: now also C?.1, C?.1, C?.1, C?.1, C?.1, C?.1, R?.1, SW?.2
- net GND: now also C?.2, C?.2, C?.2, C?.2, C?.2, C?.2, C?.2, C?.2, R?.2, SW?.1
- net at U?.22 (VCAP1): now also C?.1
- new net BOOT0: R?.1, SW?.1
- new net NRST: C?.1, R?.2, SW?.2
- no-connect marks 0 -> 2
Other:
- note added: "Bulk Decoupling Capacitor"
- note added: "Decoupling Capacitors"
- note added: "FreePill"
- note added: "Jonathan Mildon"
- note added: "MCU VCAP1"
- note added: "Reset and Boot"
- note added: "STM32F411 Open Source Development Board"
- note added: "USB C 2.0 Connection"
- moved on the sheet: F?, J?, R?
